File: a2blinky.kicad_pcb (KiCad board)
At the start: 2 copper layers, 75 x 75 mm, 25 parts, among them J1 Barrel_Jack_Switch, U1 74HC164, U2 4072, U3 AP1117-33, U4 LMC555xM

Commit message: bom
Parts:
- removed C5: 100n, Capacitor_SMD:C_0603_1608Metric
- added C8: 100n, Capacitor_SMD:C_0603_1608Metric, F.Cu at (74.9, 76.2)
- C3, C4: footprint Capacitor_SMD:C_0603_1608Metric -> Resistor_SMD:R_0603_1608Metric
- moved C6 21.6 mm to (105.4, 77.5)
- moved C7 8.98 mm to (83.8, 77.5)
Routing:
- net GND: track 51.5 -> 49.8 mm

Commit message: ecos
Parts:
- removed D1: B340, Diode_SMD:D_SMC
- added TP1: TestPoint, Connector_PinHeader_2.54mm:PinHeader_1x01_P2.54mm_Vertical, F.Cu at (96.5, 61.0)
- C1: footprint Resistor_SMD:R_0603_1608Metric -> Connector_PinHeader_2.54mm:PinHeader_1x01_P2.54mm_Horizontal
Connections:
- J1 pad 1: Net-(D1-Pad2) -> Net-(C1-Pad1)
Routing:
- net Net-(C1-Pad1): track 10.6 -> 27.0 mm, vias 0 -> 1
- net Net-(D1-Pad2): track 6.24 -> 0.00 mm
- net GND: track 49.8 -> 48.1 mm, vias 15 -> 14

Commit message: ecos
Parts:
- removed the C8 at (55.9, 76.2)
- removed Ue1: 74AHC1G04, Package_TO_SOT_SMD:SOT-353_SC-70-5
- added H1: MountingHole_Pad, MountingHole:MountingHole_3.5mm_Pad, F.Cu at (54.9, 55.2)
- added H2: MountingHole_Pad, MountingHole:MountingHole_3.5mm_Pad, F.Cu at (119.7, 56.3)
- added H3: MountingHole_Pad, MountingHole:MountingHole_3.5mm_Pad, F.Cu at (55.8, 119.1)
- added H4: MountingHole_Pad, MountingHole:MountingHole_3.5mm_Pad, F.Cu at (119.4, 119.5)
- added U5: 74AHC1G04, Package_TO_SOT_SMD:SOT-353_SC-70-5, F.Cu at (83.9, 74.9)
- C1: footprint Connector_PinHeader_2.54mm:PinHeader_1x01_P2.54mm_Horizontal -> Resistor_SMD:R_0603_1608Metric
- TP1: value TestPoint -> GND
- moved J1 5.13 mm to (64.6, 65.1)
- moved C1 0.17 mm to (82.5, 67.5)
Connections:
- net +3.3V renamed VCC
Routing:
- net Net-(C1-Pad1): track 27.0 -> 22.0 mm, vias 1 -> 0
- net VCC: track 109.2 -> 104.9 mm

Commit message: ecos
Parts:
- removed C8: 100n, Capacitor_SMD:C_0603_1608Metric
- removed U5: 74AHC1G04, Package_TO_SOT_SMD:SOT-353_SC-70-5
- U2: value 4072 -> 4002
- moved C6 32.2 mm to (75.6, 89.7)
- moved C2 29.7 mm to (86.8, 77.4), turned to 0 degrees
- moved C4 29.0 mm to (81.1, 85.6)
- moved U4 25.8 mm to (81.7, 80.0), turned to 90 degrees
- moved R2 21.7 mm to (81.7, 74.9), turned to 0 degrees
- moved D2 19.0 mm to (80.6, 112.5)
- moved D3 19.0 mm to (85.7, 112.5)
- moved D4 19.0 mm to (90.8, 112.5)
- moved D5 19.0 mm to (95.8, 112.5)
- moved R3 19.0 mm to (80.6, 107.4)
- moved R4 19.0 mm to (85.7, 107.4)
- moved R5 19.0 mm to (90.8, 107.4)
- moved R6 19.0 mm to (95.8, 107.4)
- moved R1 17.1 mm to (77.9, 74.9), turned to 0 degrees
- moved U1 16.8 mm to (78.7, 94.8), turned to 90 degrees
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Connections:
- R3 pad 1: Net-(R3-Pad1) -> Net-(U1-Pad3)
- R4 pad 1: Net-(R4-Pad1) -> Net-(U1-Pad4)
- R5 pad 1: Net-(R5-Pad1) -> Net-(U1-Pad5)
- R6 pad 1: Net-(R6-Pad1) -> Net-(U1-Pad6)
- U1 pad 10: Net-(R3-Pad1) -> unconnected-(U1-Pad10)
- U1 pad 11: Net-(R4-Pad1) -> unconnected-(U1-Pad11)
- U1 pad 12: Net-(R5-Pad1) -> unconnected-(U1-Pad12)
- U1 pad 13: Net-(R6-Pad1) -> unconnected-(U1-Pad13)
- U1 pad 3: unconnected-(U1-Pad3) -> Net-(U1-Pad3)
- U1 pad 4: unconnected-(U1-Pad4) -> Net-(U1-Pad4)
- U1 pad 5: unconnected-(U1-Pad5) -> Net-(U1-Pad5)
- U1 pad 6: unconnected-(U1-Pad6) -> Net-(U1-Pad6)
- U2 pad 1: Net-(U2-Pad1) -> Net-(U1-Pad1)
- U2 pad 2: Net-(R6-Pad1) -> Net-(U1-Pad3)
- U2 pad 3: Net-(R5-Pad1) -> Net-(U1-Pad4)
- U2 pad 4: Net-(R4-Pad1) -> Net-(U1-Pad5)
- U2 pad 5: Net-(R3-Pad1) -> Net-(U1-Pad6)
Routing:
- net Net-(R6-Pad1): track 34.9 -> 0.00 mm, vias 2 -> 0
- net Net-(R5-Pad1): track 33.6 -> 0.00 mm, vias 2 -> 0
- net Net-(R4-Pad1): track 32.3 -> 0.00 mm, vias 2 -> 0
- net Net-(R3-Pad1): track 31.1 -> 0.00 mm
- net Net-(U1-Pad6): track 0.00 -> 29.0 mm
- net Net-(U1-Pad5): track 0.00 -> 27.5 mm, vias 0 -> 2
- net Net-(U1-Pad4): track 0.00 -> 27.0 mm, vias 0 -> 2
- net Net-(U1-Pad3): track 0.00 -> 24.8 mm, vias 0 -> 2
- net Net-(U1-Pad8): track 26.8 -> 10.7 mm
- net Net-(U2-Pad1): track 12.9 -> 0.00 mm
- net VCC: track 104.9 -> 92.4 mm, vias 2 -> 0
- net Net-(U1-Pad1): track 25.0 -> 14.7 mm, vias 2 -> 0
- net GND: track 48.1 -> 41.7 mm, vias 14 -> 12
- net Net-(C4-Pad1): track 13.9 -> 10.5 mm
- net Net-(C1-Pad1): track 22.0 -> 19.8 mm

Commit message: ecos
Parts:
- added C5: 100n, Capacitor_SMD:C_0805_2012Metric, F.Cu at (76.6, 78.4)
- C1, C3, C4: footprint Resistor_SMD:R_0603_1608Metric -> Capacitor_SMD:C_0805_2012Metric
- C2, C6, C7: footprint Capacitor_SMD:C_0603_1608Metric -> Capacitor_SMD:C_0805_2012Metric
- R1, R2, R3, R4, R5, R6: footprint Resistor_SMD:R_0603_1608Metric -> Resistor_SMD:R_0805_2012Metric
- moved C6 2.13 mm to (73.9, 88.5), turned to 180 degrees
- moved R1 1.79 mm to (77.4, 73.2)
- moved C3 1.70 mm to (88.0, 67.7)
- moved R2 1.67 mm to (81.7, 73.2)
- moved C7 1.36 mm to (89.2, 88.5)
- moved C2 1.16 mm to (87.9, 77.4)
- moved C4 0.93 mm to (81.0, 86.5)
Routing:
- net GND: track 41.7 -> 31.1 mm, vias 12 -> 16
- net VCC: track 92.4 -> 98.6 mm
- net Net-(R6-Pad1): track 29.0 -> 25.3 mm
- net Net-(C4-Pad1): track 10.5 -> 13.0 mm
- net Net-(R1-Pad2): track 4.84 -> 6.93 mm
- net Net-(R5-Pad1): track 27.5 -> 25.5 mm
- net Net-(R4-Pad1): track 27.0 -> 25.1 mm
- net Net-(C2-Pad1): track 2.43 -> 3.44 mm
- net Net-(R3-Pad1): track 24.8 -> 23.8 mm
- net Net-(U1-Pad1): track 14.7 -> 15.3 mm

Commit message: silkscreen
Parts:
- added G***: LOGO, LOGO, F.Cu at (109.7, 88.4)
Other:
- board text added: "*"
- board text added: "4.6 to 12 volts"
- board text added: "GND"

Commit message: polish
Parts:
- added J2: Conn_01x02_Male, Connector_PinHeader_2.54mm:PinHeader_1x02_P2.54mm_Vertical, F.Cu at (61.9, 79.8)
- moved G*** 2.07 mm to (109.1, 90.4)
Routing:
- net Net-(C1-Pad1): track 19.7 -> 36.0 mm
Other:
- board text added: "+"
Changed lines of the file:
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@@
     )
   )
+  (footprint "Connector_PinHeader_2.54mm:PinHeader_1x02_P2.54mm_Vertical" (layer "F.Cu")
+    (at 61.9 79.8)
+    (descr "Through hole straight pin header, 1x02, 2.54mm pitch, single row")
+    (tags "Through hole pin header THT 1x02 2.54mm single row")
+    (property "Sheetfile" "a2blinky.kicad_sch")
+    (property "Sheetname" "")
+    (attr through_hole)
+    (fp_text reference "J2" (at 0 -2.33) (layer "F.SilkS")
+      (effects (font (size 1 1) (thickness 0.15)))
+    )
+    (fp_text value "Conn_01x02_Male" (at 0 4.87) (layer "F.Fab")
+      (effects (font (size 1 1) (thickness 0.15)))
+    )
+    (fp_text user "${REFERENCE}" (at 0 1.27 90) (layer "F.Fab")
+      (effects (font (size 1 1) (thickness 0.15)))
+    )
+    (fp_line (start -1.33 1.27) (end -1.33 3.87) (layer "F.SilkS") (width 0.12))
+    (fp_line (start -1.33 -1.33) (end 0 -1.33) (layer "F.SilkS") (width 0.12))
+    (fp_line (start -1.33 3.87) (end 1.33 3.87) (layer "F.SilkS") (width 0.12))
+    (fp_line (start -1.33 0) (end -1.33 -1.33) (layer "F.SilkS") (width 0.12))
+    (fp_line (start -1.33 1.27) (end 1.33 1.27) (layer "F.SilkS") (width 0.12))
+    (fp_line (start 1.33 1.27) (end 1.33 3.87) (layer "F.SilkS") (width 0.12))
+    (fp_line (start -1.8 4.35) (end 1.8 4.35) (layer "F.CrtYd") (width 0.05))
+    (fp_line (start 1.8 -1.8) (end -1.8 -1.8) (layer "F.CrtYd") (width 0.05))
+    (fp_line (start 1.8 4.35) (end 1.8 -1.8) (layer "F.CrtYd") (width 0.05))
+    (fp_line (start -1.8 -1.8) (end -1.8 4.35) (layer "F.CrtYd") (width 0.05))
+    (fp_line (start 1.27 -1.27) (end 1.27 3.81) (layer "F.Fab") (width 0.1))
+    (fp_line (start -0.635 -1.27) (end 1.27 -1.27) (layer "F.Fab") (width 0.1))
+    (fp_line (start 1.27 3.81) (end -1.27 3.81) (layer "F.Fab") (width 0.1))
+    (fp_line (start -1.27 -0.635) (end -0.635 -1.27) (layer "F.Fab") (width 0.1))
+    (fp_line (start -1.27 3.81) (end -1.27 -0.635) (layer "F.Fab") (width 0.1))
+    (pad "1" thru_hole rect (at 0 0) (size 1.7 1.7) (drill 1) (layers *.Cu *.Mask)
+      (net 1 "Net-(C1-Pad1)") (pinfunction "Pin_1") (pintype "passive"))
+    (pad "2" thru_hole oval (at 0 2.54) (size 1.7 1.7) (drill 1) (layers *.Cu *.Mask)
+      (net 2 "GND") (pinfunction "Pin_2") (pintype "passive"))
+    (model "${KICAD6_3DMODEL_DIR}/Connector_PinHeader_2.54mm.3dshapes/PinHeader_1x02_P2.54mm_Vertical.wrl"
+      (offset (xyz 0 0 0))
+      (scale (xyz 1 1 1))
+      (rotate (xyz 0 0 0))
+    )
+  )
   (footprint "Resistor_SMD:R_0805_2012Metric" (layer "F.Cu")
     (at 77.37 73.17)
@@
   )
   (footprint "LOGO" (layer "F.Cu")
-    (at 109.68 88.41 90)
+    (at 109.1 90.4 90)
     (attr board_only exclude_from_pos_files exclude_from_bom)
-    (fp_text reference "G***" (at 0 0 90) (layer "F.SilkS")
+    (fp_text reference "G***" (at 0 0 90) (layer "F.SilkS") hide
       (effects (font (size 1.524 1.524) (thickness 0.3)))
     )
@@
   (gr_line (start 50 125) (end 50 50) (layer "Edge.Cuts") (width 0.1))
   (gr_line (start 50 50) (end 125 50) (layer "Edge.Cuts") (width 0.1))
+  (gr_text "+" (at 58.3 79.5) (layer "F.Cu")
+    (effects (font (size 1.5 1.5) (thickness 0.3)))
+  )
   (gr_text "*" (at 87.2 99.4) (layer "F.SilkS")
     (effects (font (size 1 1) (thickness 0.15)))
@@
     (effects (font (size 1 1) (thickness 0.15)))
   )
+  (segment (start 62.8 79.8) (end 64.63 77.97) (width 0.25) (layer "F.Cu") (net 1))
+  (segment (start 61.9 79.8) (end 62.8 79.8) (width 0.25) (layer "F.Cu") (net 1))
   (segment (start 75.76 63.26) (end 83.21 63.26) (width 0.25) (layer "F.Cu") (net 1))
   (segment (start 73.45 65.57) (end 75.76 63.26) (width 0.25) (layer "F.Cu") (net 1))
   (segment (start 73.0125 65.1325) (end 73.45 65.57) (width 0.25) (layer "F.Cu") (net 1))
+  (segment (start 64.63 77.97) (end 64.63 65.1325) (width 0.25) (layer "F.Cu") (net 1))
   (segment (start 64.63 65.1325) (end 73.0125 65.1325) (width 0.25) (layer "F.Cu") (net 1))
   (segment (start 87.05 67.71) (end 85.06 67.71) (width 0.25) (layer "F.Cu") (net 2))
