File: a2blinky.kicad_sch (KiCad schematic)
At the start: 25 parts, among them J1 Barrel_Jack_Switch, U1 74HC164, U2 4072, U3 AP1117-33, U4 LMC555xM

Commit message: bom
Parts:
- removed C5: 100n, Capacitor_SMD:C_0603_1608Metric, symbol Device:C_Small
- C1: LCSC (none) -> C96446
- C2, C6, C7, C8: LCSC (none) -> C14663
- C3, C4: footprint Capacitor_SMD:C_0603_1608Metric -> Resistor_SMD:R_0603_1608Metric; LCSC (none) -> C96446
- D1: LCSC (none) -> C64982
- D2, D3, D4, D5: LCSC (none) -> C2297
- J1: LCSC (none) -> C194407
- R1, R2, R3, R4, R5, R6: LCSC (none) -> C25197
- U1: LCSC (none) -> C6825
- U2: LCSC (none) -> C68527
- U3: LCSC (none) -> C6186
- U4: LCSC (none) -> C90760
- Ue1: LCSC (none) -> C7466

Commit message: ecos
Parts:
- removed D1: B340, Diode_SMD:D_SMC, symbol Diode:B340
- added H1, H2, H3, H4: MountingHole_Pad, symbol Mechanical:MountingHole_Pad
- added TP1: TestPoint, Connector_PinHeader_2.54mm:PinHeader_1x01_P2.54mm_Vertical, symbol Connector:TestPoint
- C1: footprint Resistor_SMD:R_0603_1608Metric -> MountingHole:MountingHole_3.5mm_Pad
Connections:
- net GND: now also H1.1, H2.1, H3.1, H4.1, TP1.1
- net at C1.1, U3.3 (VI): now also J1.1

Commit message: ecos
Parts:
- removed Ue1: 74AHC1G04, Package_TO_SOT_SMD:SOT-353_SC-70-5, symbol 74xGxx:74AHC1G04
- added U5: 74AHC1G04, Package_TO_SOT_SMD:SOT-353_SC-70-5, symbol 74xGxx:74AHC1G04
- C1: footprint MountingHole:MountingHole_3.5mm_Pad -> Resistor_SMD:R_0603_1608Metric
- H1, H2, H3, H4: footprint (none) -> MountingHole:MountingHole_3.5mm_Pad
- TP1: value TestPoint -> GND
Connections:
- net GND: now also U5.3 (GND)
- net at U1.1 (DSA), U1.2 (DSB): now also U5.4
- net at U2.1: now also U5.2
- net +3.3V renamed VCC
- net VCC: now also U5.5 (VCC)
- no-connect marks 1 -> 5

Commit message: ecos
Parts:
- removed C8: 100n, Capacitor_SMD:C_0603_1608Metric, symbol Device:C_Small
- removed U2: 4072, Package_SO:SOIC-14_3.9x8.7mm_P1.27mm, symbol 4xxx:4072
- removed U5: 74AHC1G04, Package_TO_SOT_SMD:SOT-353_SC-70-5, symbol 74xGxx:74AHC1G04
- added U2: 4002, symbol 4xxx:4002
Connections:
- net GND: now also U2.10, U2.11, U2.12, U2.7 (VSS), U2.9
- net VCC: now also U2.14 (VDD)
- net at U1.1 (DSA), U1.2 (DSB): now also U2.1
- net at U1.10 (Q4): no longer R3.1
- net at U1.11 (Q5): no longer R4.1
- net at U1.12 (Q6): no longer R5.1
- net at U1.13 (Q7): no longer R6.1
- net at U1.3 (Q0): now also R3.1, U2.2
- net at U1.4 (Q1): now also R4.1, U2.3
- net at U1.5 (Q2): now also R5.1, U2.4
- net at U1.6 (Q3): now also R6.1, U2.5
Other:
- moved on the sheet: D2, D3, D4, D5, R3, R4, R5, R6

Commit message: ecos
Parts:
- added C5: 100n, Capacitor_SMD:C_0805_2012Metric, symbol Device:C_Small
- C1, C3, C4: footprint Resistor_SMD:R_0603_1608Metric -> Capacitor_SMD:C_0805_2012Metric; LCSC C96446 -> C15850
- C2, C6, C7: footprint Capacitor_SMD:C_0603_1608Metric -> Capacitor_SMD:C_0805_2012Metric; LCSC C14663 -> C49678
- R1, R2, R3, R4, R5, R6: footprint Resistor_SMD:R_0603_1608Metric -> Resistor_SMD:R_0805_2012Metric; LCSC C25197 -> C17414
- U2: footprint (none) -> Package_SO:SOIC-14_3.9x8.7mm_P1.27mm
Connections:
- net GND: now also C5.2
- net VCC: now also C5.1

Commit message: polish
Parts:
- added J2: Conn_01x02_Male, Connector_PinHeader_2.54mm:PinHeader_1x02_P2.54mm_Vertical, symbol Connector:Conn_01x02_Male
Connections:
- net GND: now also J2.2 (Pin_2)
- net at C1.1, J1.1, U3.3 (VI): now also J2.1 (Pin_1)
Other:
- note added: "4.6 to 12 volts"
Changed lines of the file:
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@@
   (junction (at 162.56 115.57) (diameter 0) (color 0 0 0 0)
+  )
+  (junction (at 48.26 35.56) (diameter 0) (color 0 0 0 0)
   )
   (junction (at 156.21 67.31) (diameter 0) (color 0 0 0 0)
@@
     (stroke (width 0) (type default) (color 0 0 0 0))
   )
-  (wire (pts (xy 44.45 35.56) (xy 54.61 35.56))
+  (wire (pts (xy 44.45 35.56) (xy 48.26 35.56))
     (stroke (width 0) (type default) (color 0 0 0 0))
   )
@@
     (stroke (width 0) (type default) (color 0 0 0 0))
   )
+  (wire (pts (xy 34.29 58.42) (xy 48.26 58.42))
+    (stroke (width 0) (type default) (color 0 0 0 0))
+  )
   (wire (pts (xy 214.63 67.31) (xy 214.63 69.85))
     (stroke (width 0) (type default) (color 0 0 0 0))
@@
     (stroke (width 0) (type default) (color 0 0 0 0))
   )
+  (wire (pts (xy 48.26 35.56) (xy 54.61 35.56))
+    (stroke (width 0) (type default) (color 0 0 0 0))
+  )
   (wire (pts (xy 67.31 44.45) (xy 67.31 43.18))
     (stroke (width 0) (type default) (color 0 0 0 0))
@@
     (stroke (width 0) (type default) (color 0 0 0 0))
   )
+  (wire (pts (xy 48.26 58.42) (xy 48.26 35.56))
+    (stroke (width 0) (type default) (color 0 0 0 0))
+  )
   (wire (pts (xy 209.55 74.93) (xy 214.63 74.93))
     (stroke (width 0) (type default) (color 0 0 0 0))
@@
   (wire (pts (xy 105.41 105.41) (xy 105.41 92.71))
     (stroke (width 0) (type default) (color 0 0 0 0))
+  )
+  (text "4.6 to 12 volts" (at 22.86 73.66 0)
+    (effects (font (size 1.27 1.27)) (justify left bottom))
   )
   (symbol (lib_id "Device:LED_Small") (at 207.01 69.85 180) (unit 1)
@@
     (pin "2")
   )
+  (symbol (lib_id "Connector:Conn_01x02_Male") (at 29.21 58.42 0) (unit 1)
+    (in_bom yes) (on_board yes) (fields_autoplaced)
+    (property "Reference" "J2" (id 0) (at 29.845 53.34 0))
+    (property "Value" "Conn_01x02_Male" (id 1) (at 29.845 55.88 0))
+    (property "Footprint" "Connector_PinHeader_2.54mm:PinHeader_1x02_P2.54mm_Vertical" (id 2) (at 29.21 58.42 0)
+      (effects (font (size 1.27 1.27)) hide)
+    )
+    (property "Datasheet" "~" (id 3) (at 29.21 58.42 0)
+      (effects (font (size 1.27 1.27)) hide)
+    )
+    (pin "1")
+    (pin "2")
+  )
   (symbol (lib_id "power:PWR_FLAG") (at 96.52 36.83 0) (unit 1)
     (in_bom yes) (on_board yes) (fields_autoplaced)
@@
     (pin "2")
   )
+  (symbol (lib_id "power:GND") (at 34.29 60.96 0) (unit 1)
+    (in_bom yes) (on_board yes) (fields_autoplaced)
+    (property "Reference" "#PWR05" (id 0) (at 34.29 67.31 0)
+      (effects (font (size 1.27 1.27)) hide)
+    )
+    (property "Value" "GND" (id 1) (at 34.29 66.04 0))
+    (property "Footprint" "" (id 2) (at 34.29 60.96 0)
+      (effects (font (size 1.27 1.27)) hide)
+    )
+    (property "Datasheet" "" (id 3) (at 34.29 60.96 0)
+      (effects (font (size 1.27 1.27)) hide)
+    )
+    (pin "1")
+  )
   (symbol (lib_id "power:GND") (at 91.44 97.79 0) (unit 1)
     (in_bom yes) (on_board yes) (fields_autoplaced)
@@
       (reference "#PWR04") (unit 1) (value "GND") (footprint "")
     )
+    (path "/ed183389-67f1-4303-bc85-bd462356c65f"
+      (reference "#PWR05") (unit 1) (value "GND") (footprint "")
+    )
     (path "/7898eff3-f537-48d1-935b-aa5ace8bdf9c"
       (reference "#PWR06") (unit 1) (value "GND") (footprint "")
@@
       (reference "J1") (unit 1) (value "Barrel_Jack_Switch") (footprint "Connector_BarrelJack:BarrelJack_Horizontal")
     )
+    (path "/81aa642b-6bdd-4eed-9f8d-b277e8a8ae19"
+      (reference "J2") (unit 1) (value "Conn_01x02_Male") (footprint "Connector_PinHeader_2.54mm:PinHeader_1x02_P2.54mm_Vertical")
+    )
     (path "/8127e4e8-8832-46b2-ada7-acde11994f72"

Commit message: step3
Parts:
- renumbered C3 to C2, C2 to C3, C6 to C5, C7 to C6, C5 to C7, D2 to D1, D3 to D2, D4 to D3, D5 to D4, U3 to U1, U4 to U3, U1 to U4
Other:
- moved on the sheet: C1, C2, C3, C4, C5, C6, C7, D1, D2, D3, D4, H1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
